Commit message: adapting FoV

File: urdf/realsense-D435.macro.xacro (robot description, xacro)
@@ -15,5 +15,5 @@
     <link name="${prefix}D435_camera">
         <visual>
-            <origin rpy="0 0 0" xyz="0 0 0"/>
+            <origin rpy="${pi/2} 0 ${pi/2}" xyz="0 0 0"/>
             <geometry>
                 <mesh filename="package://realsense_gazebo_plugin/models/realsense_camera/meshes/realsense_d435.stl"/>
@@ -104,5 +104,5 @@
             <clip>
                 <near>0.1</near>
-                <far>100</far>
+                <far>7</far> <!-- to mimic depth cam view -->
             </clip>
             <noise>
@@ -114,5 +114,5 @@
             <always_on>1</always_on>
             <update_rate>60</update_rate>
-            <visualize>0</visualize>
+            <visualize>1</visualize>
         </sensor>
         <sensor name="ired1" type="camera">
@@ -172,5 +172,5 @@
             <clip>
                     <near>0.1</near>
-                    <far>100</far>
+                    <far>7</far>
             </clip>
             <noise>
